File: wave-cover/wave-cover.kicad_pcb (KiCad board)
At the start: 2 copper layers, 60 x 60 mm, 11 parts

Commit message: Refresh
Parts:
- H108, H109: value MountingHole_2mm_Pad_2.4mm -> MountingHole_10mm
Changed lines of the file:
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@@
     (property "ki_description" "Mounting Hole with connection")
     (property "ki_keywords" "mounting hole")
+    (attr exclude_from_bom)
     (fp_text reference "H101" (at 0 -4 unlocked) (layer "F.SilkS") hide
         (effects (font (size 1 1) (thickness 0.15)))
@@
         (effects (font (size 1 1) (thickness 0.15)))
     )
-    (fp_text value "MountingHole_2mm_Pad_2.4mm" (at 0 7.5) (layer "F.Fab") hide
+    (fp_text value "MountingHole_10mm" (at 0 7.5) (layer "F.Fab") hide
         (effects (font (size 1 1) (thickness 0.15)))
     )
@@
     (property "ki_description" "Mounting Hole with connection")
     (property "ki_keywords" "mounting hole")
+    (attr exclude_from_bom)
     (fp_text reference "H104" (at 0 -4 unlocked) (layer "F.SilkS") hide
         (effects (font (size 1 1) (thickness 0.15)))
@@
         (effects (font (size 1 1) (thickness 0.15)))
     )
-    (fp_text value "MountingHole_2mm_Pad_2.4mm" (at 0 7.5) (layer "F.Fab") hide
+    (fp_text value "MountingHole_10mm" (at 0 7.5) (layer "F.Fab") hide
         (effects (font (size 1 1) (thickness 0.15)))
     )
@@
     (property "ki_description" "Mounting Hole with connection")
     (property "ki_keywords" "mounting hole")
+    (attr exclude_from_bom)
     (fp_text reference "H102" (at 0 -4 unlocked) (layer "F.SilkS") hide
         (effects (font (size 1 1) (thickness 0.15)))
@@
     (property "ki_description" "Mounting Hole with connection")
     (property "ki_keywords" "mounting hole")
+    (attr exclude_from_bom)
     (fp_text reference "H103" (at 0 -4 unlocked) (layer "F.SilkS") hide
         (effects (font (size 1 1) (thickness 0.15)))
