File: wave-cover/wave-cover.kicad_sch (KiCad schematic)
At the start: 11 parts

Commit message: Refresh
Parts:
- H108, H109: value MountingHole_2mm_Pad_2.4mm -> MountingHole_10mm
Changed lines of the file:
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@@
-    (stroke (width 0) (type default))
-  )
-  (wire (pts (xy 161.29 73.66) (xy 161.29 85.09))
     (stroke (width 0) (type default))
   )
@@
         (path "/6c8448b4-b04d-47e1-934e-e40cbe27a7be"
           (reference "H102") (unit 1)
-        )
-      )
-    )
-  )
-  (symbol (lib_id "power:GND") (at 161.29 85.09 0) (unit 1)
-    (in_bom yes) (on_board yes) (dnp no) (fields_autoplaced)
-    (property "Reference" "#PWR0102" (at 161.29 91.44 0)
-      (effects (font (size 1.27 1.27)) hide)
-    )
-    (property "Value" "GND" (at 161.29 90.17 0)
-      (effects (font (size 1.27 1.27)))
-    )
-    (property "Footprint" "" (at 161.29 85.09 0)
-      (effects (font (size 1.27 1.27)) hide)
-    )
-    (property "Datasheet" "" (at 161.29 85.09 0)
-      (effects (font (size 1.27 1.27)) hide)
-    )
-    (pin "1")
-    (instances
-      (project "wave-cover"
-        (path "/6c8448b4-b04d-47e1-934e-e40cbe27a7be"
-          (reference "#PWR0102") (unit 1)
         )
       )
@@
       (effects (font (size 1.27 1.27)) (justify left))
     )
-    (property "Value" "MountingHole_2mm_Pad_2.4mm" (at 166.37 75.565 90)
+    (property "Value" "MountingHole_10mm" (at 166.37 75.565 90)
       (effects (font (size 1.27 1.27)) (justify left))
     )
@@
       (effects (font (size 1.27 1.27)) (justify left))
     )
-    (property "Value" "MountingHole_2mm_Pad_2.4mm" (at 166.37 83.185 90)
+    (property "Value" "MountingHole_10mm" (at 166.37 83.185 90)
       (effects (font (size 1.27 1.27)) (justify left))
     )
