File: AmplifierAudio.kicad_sch (KiCad schematic)
At the start: 50 parts, among them Q201 IRF9358, U201 MA12070P

Commit message: Refresh
Other:
- moved on the sheet: D201, D202
Changed lines of the file:
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@@
   (junction (at 101.6 167.64) (diameter 0) (color 0 0 0 0)
   )
-  (junction (at 189.23 80.01) (diameter 0) (color 0 0 0 0)
-  )
   (junction (at 119.38 134.62) (diameter 0) (color 0 0 0 0)
+  )
+  (junction (at 189.23 81.28) (diameter 0) (color 0 0 0 0)
   )
   (no_connect (at 91.44 114.3))
@@
     (stroke (width 0) (type default))
   )
+  (wire (pts (xy 189.23 81.28) (xy 189.23 83.82))
+    (stroke (width 0) (type default))
+  )
   (wire (pts (xy 29.21 129.54) (xy 91.44 129.54))
     (stroke (width 0) (type default))
@@
     (stroke (width 0) (type default))
   )
-  (wire (pts (xy 189.23 80.01) (xy 189.23 83.82))
-    (stroke (width 0) (type default))
-  )
   (wire (pts (xy 137.16 149.86) (xy 148.59 149.86))
     (stroke (width 0) (type default))
@@
     (stroke (width 0) (type default))
   )
-  (wire (pts (xy 176.53 80.01) (xy 184.15 80.01))
+  (wire (pts (xy 176.53 81.28) (xy 184.15 81.28))
     (stroke (width 0) (type default))
   )
@@
     (effects (font (size 1.27 1.27)) (justify left bottom))
   )
-  (label "PVDD" (at 176.53 80.01 0) (fields_autoplaced)
+  (label "PVDD" (at 176.53 81.28 0) (fields_autoplaced)
     (effects (font (size 1.27 1.27)) (justify left bottom))
   )
@@
     )
   )
-  (symbol (lib_id "V2_Diode:PMEG3010ER") (at 186.69 80.01 0) (unit 1)
-    (in_bom yes) (on_board yes) (dnp no)
-    (property "Reference" "D201" (at 176.53 72.39 0)
-      (effects (font (size 1.27 1.27)) (justify left))
-    )
-    (property "Value" "PMEG3010ER" (at 176.53 74.93 0)
-      (effects (font (size 1.27 1.27)) (justify left))
-    )
-    (property "Footprint" "Diode_SMD:Nexperia_CFP3_SOD-123W" (at 186.69 84.455 0)
-      (effects (font (size 1.27 1.27)) hide)
-    )
-    (property "Datasheet" "" (at 186.69 80.01 0)
+  (symbol (lib_id "V2_Diode:PMEG3010ER") (at 186.69 81.28 0) (unit 1)
+    (in_bom yes) (on_board yes) (dnp no)
+    (property "Reference" "D201" (at 176.53 73.66 0)
+      (effects (font (size 1.27 1.27)) (justify left))
+    )
+    (property "Value" "PMEG3010ER" (at 176.53 76.2 0)
+      (effects (font (size 1.27 1.27)) (justify left))
+    )
+    (property "Footprint" "Diode_SMD:Nexperia_CFP3_SOD-123W" (at 186.69 85.725 0)
+      (effects (font (size 1.27 1.27)) hide)
+    )
+    (property "Datasheet" "" (at 186.69 81.28 0)
       (effects (font (size 1.27 1.27)) hide)
     )
@@
     )
   )
-  (symbol (lib_id "power:GND") (at 194.31 80.01 90) (unit 1)
-    (in_bom yes) (on_board yes) (dnp no)
-    (property "Reference" "#PWR0206" (at 200.66 80.01 0)
-      (effects (font (size 1.27 1.27)) hide)
-    )
-    (property "Value" "GND" (at 199.39 80.01 90)
-      (effects (font (size 1.27 1.27)))
-    )
-    (property "Footprint" "" (at 194.31 80.01 0)
-      (effects (font (size 1.27 1.27)) hide)
-    )
-    (property "Datasheet" "" (at 194.31 80.01 0)
+  (symbol (lib_id "power:GND") (at 194.31 81.28 90) (unit 1)
+    (in_bom yes) (on_board yes) (dnp no)
+    (property "Reference" "#PWR0206" (at 200.66 81.28 0)
+      (effects (font (size 1.27 1.27)) hide)
+    )
+    (property "Value" "GND" (at 199.39 81.28 90)
+      (effects (font (size 1.27 1.27)))
+    )
+    (property "Footprint" "" (at 194.31 81.28 0)
+      (effects (font (size 1.27 1.27)) hide)
+    )
+    (property "Datasheet" "" (at 194.31 81.28 0)
       (effects (font (size 1.27 1.27)) hide)
     )
@@
     )
   )
-  (symbol (lib_id "V2_Diode:PMEG3010ER") (at 191.77 80.01 0) (unit 1)
-    (in_bom yes) (on_board yes) (dnp no)
-    (property "Reference" "D202" (at 190.5 72.39 0)
-      (effects (font (size 1.27 1.27)) (justify left))
-    )
-    (property "Value" "PMEG3010ER" (at 190.5 74.93 0)
-      (effects (font (size 1.27 1.27)) (justify left))
-    )
-    (property "Footprint" "Diode_SMD:Nexperia_CFP3_SOD-123W" (at 191.77 84.455 0)
-      (effects (font (size 1.27 1.27)) hide)
-    )
-    (property "Datasheet" "" (at 191.77 80.01 0)
-      (effects (font (size 1.27 1.27)) hide)
-    )
+  (symbol (lib_id "V2_Diode:PMEG3010ER") (at 191.77 81.28 0) (unit 1)
+    (in_bom yes) (on_board yes) (dnp no)
+    (property "Reference" "D202" (at 190.5 73.66 0)
+      (effects (font (size 1.27 1.27)) (justify left))
+    )
+    (property "Value" "PMEG3010ER" (at 190.5 76.2 0)
+      (effects (font (size 1.27 1.27)) (justify left))
+    )
+    (property "Footprint" "Diode_SMD:Nexperia_CFP3_SOD-123W" (at 191.77 85.725 0)
+      (effects (font (size 1.27 1.27)) hide)
+    )
+    (property "Datasheet" "" (at 191.77 81.28 0)
+      (effects (font (size 1.27 1.27)) hide)
+    )

Commit message: Update to Kicad 8
Parts:
- renumbered R103 to R201, R103 to R202, R103 to R203

Commit message: Refresh
Parts:
- renumbered C233 to C207, C207 to C208, C208 to C209, C232 to C210, C209 to C211, C210 to C212, C211 to C213, C212 to C214, C213 to C215, C214 to C216, C215 to C217, C216 to C218, C217 to C219, C218 to C220, C219 to C221, C220 to C222, C221 to C223, C222 to C224, C223 to C225, C224 to C226, C225 to C227, C226 to C228, C227 to C229, C228 to C230, C229 to C231, C230 to C232, C231 to C233
Other:
- moved on the sheet: C210, R201, R202, R203
