File: LEDStrip.kicad_sch (KiCad schematic)
At the start: 3 parts, among them J501 WAGO-2065, J502 WAGO-2065, U501 74AHC1G125

Commit message: Refresh
Changed lines of the file:
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@@
 (kicad_sch
-	(version 20231120)
+	(version 20250114)
 	(generator "eeschema")
-	(generator_version "8.0")
+	(generator_version "9.0")
 	(paper "A4")
 	(title_block
@@
 	(label "WS2812-data"
 		(at 146.05 111.76 0)
-		(fields_autoplaced yes)
 		(effects
 			(font
@@
 		(shape input)
 		(at 121.92 111.76 180)
-		(fields_autoplaced yes)
 		(effects
 			(font
@@
 		(at 175.26 109.22 0)
 		(unit 1)
-		(exclude_from_sim yes)
+		(exclude_from_sim no)
 		(in_bom yes)
 		(on_board yes)
@@
 		(at 175.26 111.76 0)
 		(unit 1)
-		(exclude_from_sim yes)
+		(exclude_from_sim no)
 		(in_bom yes)
 		(on_board yes)
