File: LinkPlug.kicad_sch (KiCad schematic)
At the start: 6 parts, among them J301 2x05_Horizontal, U301 SN65MLVD203B

Commit message: Refresh
Parts:
- removed R301, R303: 10k, Resistor_SMD:R_0603_1608Metric, symbol Device:R_Small
- U301: value SN65MLVD203B -> THVD24x2; footprint V2_Package_DFN_QFN:WQFN-16-1EP_4x4mm_P0.65mm_EP2.7x2.7mm_ThermalVias -> V2_Package_SON:VSON-10-4-1EP_3x3mm_P0.5mm_EP1.65x2.4mm_ThermalVias; symbol V2_Interface_LVDS:SN65MLVD203B -> V2_Interface_RS485:THVD24x2
- renumbered R302 to R301
Connections:
- net +3V3: now also U301.10 (VCC); no longer U301.13 (VCC), U301.14 (VCC)
- net GND: now also U301.11 (GND); no longer U301.17 (GND), U301.6 (GND)
- net RX-A: now also U301.9 (A); no longer U301.12 (A)
- net RX-B: now also U301.8 (B); no longer U301.11 (B)
- net TX-Y: now also U301.6 (Y); no longer U301.9 (Y)
- net TX-Z: now also U301.7 (Z); no longer U301.10 (Z)
