File: LinkSocket.kicad_sch (KiCad schematic)
At the start: 6 parts, among them J401 2x05_Horizontal, U401 SN65MLVD203B

Commit message: Refresh
Parts:
- removed R401, R403: 10k, Resistor_SMD:R_0603_1608Metric, symbol Device:R_Small
- U401: value SN65MLVD203B -> THVD24x2; footprint V2_Package_DFN_QFN:WQFN-16-1EP_4x4mm_P0.65mm_EP2.7x2.7mm_ThermalVias -> V2_Package_SON:VSON-10-4-1EP_3x3mm_P0.5mm_EP1.65x2.4mm_ThermalVias; symbol V2_Interface_LVDS:SN65MLVD203B -> V2_Interface_RS485:THVD24x2
- renumbered R402 to R401
Connections:
- net +3V3: now also U401.10 (VCC); no longer U401.13 (VCC), U401.14 (VCC)
- net GND: now also U401.11 (GND); no longer U401.17 (GND), U401.6 (GND)
- net RX-A: now also U401.9 (A); no longer U401.12 (A)
- net RX-B: now also U401.8 (B); no longer U401.11 (B)
- net TX-Y: now also U401.6 (Y); no longer U401.9 (Y)
- net TX-Z: now also U401.7 (Z); no longer U401.10 (Z)
