File: wave.kicad_sch (KiCad schematic)
At the start: 64 parts, among them J101 CORTEX-DEBUG, J102 WAGO-2065, J103 WAGO-2065, J104 WAGO-2065, J105 WAGO-2065, J106 WAGO-2065, J107 WAGO-2065, SW101 SW_Push, SW102 SW_Push, U101 TPS78433QWDRBRQ1, U102 ATSAMD51J, Y101 32k768

Commit message: Refresh
Parts:
- added ICON110: Dot, V2_Artwork:Dot_Small, symbol V2_Artwork:Dot
- added ICON111: Plug, V2_Artwork:Plug_Small, symbol V2_Artwork:Plug
- added ICON112: Socket, V2_Artwork:Socket_Small, symbol V2_Artwork:Socket
- R103, R104: value 5k1 -> 2k7
Other:
- moved on the sheet: ICON103, ICON107, ICON108
Changed lines of the file:
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@@
   (title_block
     (title "V2 wave")
-    (date "2023-06-01")
-    (rev "1")
+    (date "2023-07-10")
+    (rev "2")
     (company "Versio Duo")
     (comment 1 "Power Amplifier")
@@
     (stroke (width 0) (type default))
   )
-  (wire (pts (xy 34.29 148.59) (xy 59.69 148.59))
-    (stroke (width 0) (type default))
-  )
   (wire (pts (xy 67.31 127) (xy 69.85 127))
     (stroke (width 0) (type default))
@@
     (stroke (width 0) (type default))
   )
+  (wire (pts (xy 34.29 148.59) (xy 59.69 148.59))
+    (stroke (width 0) (type default))
+  )
   (wire (pts (xy 22.86 176.53) (xy 22.86 173.99))
     (stroke (width 0) (type default))
@@
     (effects (font (size 1.27 1.27)) (justify left bottom))
   )
-  (label "Supply +24V" (at 35.56 148.59 0) (fields_autoplaced)
+  (label "Supply +24V" (at 36.83 148.59 0) (fields_autoplaced)
     (effects (font (size 1.27 1.27)) (justify left bottom))
   )
@@
     )
   )
-  (symbol (lib_id "V2_Artwork:Plus") (at 248.92 142.24 0) (unit 1)
+  (symbol (lib_id "V2_Artwork:Plus") (at 217.17 142.24 0) (unit 1)
     (in_bom no) (on_board yes) (dnp no) (fields_autoplaced)
-    (property "Reference" "ICON103" (at 251.46 142.875 0)
+    (property "Reference" "ICON103" (at 219.71 142.875 0)
       (effects (font (size 1.27 1.27)) (justify left))
     )
-    (property "Value" "Plus" (at 246.38 147.32 0)
+    (property "Value" "Plus" (at 214.63 147.32 0)
       (effects (font (size 1.27 1.27)) (justify left bottom) hide)
     )
-    (property "Footprint" "V2_Artwork:Plus_Small" (at 248.92 149.86 0)
+    (property "Footprint" "V2_Artwork:Plus_Small" (at 217.17 149.86 0)
       (effects (font (size 1.27 1.27)) hide)
     )
-    (property "Datasheet" "" (at 248.92 142.24 0)
+    (property "Datasheet" "" (at 217.17 142.24 0)
       (effects (font (size 1.27 1.27)) hide)
     )
-    (property "Sim.Enable" "0" (at 248.92 142.24 0)
+    (property "Sim.Enable" "0" (at 217.17 142.24 0)
       (effects (font (size 1.27 1.27)) hide)
     )
@@
       (effects (font (size 1.27 1.27)) (justify left))
     )
-    (property "Value" "5k1" (at 79.375 171.45 0)
+    (property "Value" "2k7" (at 79.375 171.45 0)
       (effects (font (size 1.27 1.27)) (justify left))
     )
@@
     )
   )
+  (symbol (lib_id "V2_Artwork:Plug") (at 182.88 147.32 0) (unit 1)
+    (in_bom no) (on_board yes) (dnp no) (fields_autoplaced)
+    (property "Reference" "ICON111" (at 185.42 147.32 0)
+      (effects (font (size 1.27 1.27)) (justify left))
+    )
+    (property "Value" "Plug" (at 180.34 152.4 0)
+      (effects (font (size 1.27 1.27)) (justify left bottom) hide)
+    )
+    (property "Footprint" "V2_Artwork:Plug_Small" (at 182.88 154.94 0)
+      (effects (font (size 1.27 1.27)) hide)
+    )
+    (property "Datasheet" "" (at 182.7022 147.32 0)
+      (effects (font (size 1.27 1.27)) hide)
+    )
+    (property "Sim.Enable" "0" (at 182.88 147.32 0)
+      (effects (font (size 1.27 1.27)) hide)
+    )
+    (instances
+      (project "wave"
+        (path "/6c8448b4-b04d-47e1-934e-e40cbe27a7be"
+          (reference "ICON111") (unit 1)
+        )
+      )
+    )
+  )
   (symbol (lib_id "V2_Mechanical:MountingHole_3mm") (at 256.54 176.53 0) (unit 1)
     (in_bom no) (on_board yes) (dnp no)
@@
     )
   )
-  (symbol (lib_id "V2_Artwork:Plus") (at 248.92 147.32 0) (unit 1)
+  (symbol (lib_id "V2_Artwork:Plus") (at 248.92 142.24 0) (unit 1)
     (in_bom no) (on_board yes) (dnp no) (fields_autoplaced)
-    (property "Reference" "ICON107" (at 251.46 147.955 0)
+    (property "Reference" "ICON107" (at 251.46 142.875 0)
       (effects (font (size 1.27 1.27)) (justify left))
     )
-    (property "Value" "Plus" (at 246.38 152.4 0)
+    (property "Value" "Plus" (at 246.38 147.32 0)
       (effects (font (size 1.27 1.27)) (justify left bottom) hide)
     )
-    (property "Footprint" "V2_Artwork:Plus_Small" (at 248.92 154.94 0)
+    (property "Footprint" "V2_Artwork:Plus_Small" (at 248.92 149.86 0)
       (effects (font (size 1.27 1.27)) hide)
     )
-    (property "Datasheet" "" (at 248.92 147.32 0)
+    (property "Datasheet" "" (at 248.92 142.24 0)
       (effects (font (size 1.27 1.27)) hide)
     )
-    (property "Sim.Enable" "0" (at 248.92 147.32 0)
+    (property "Sim.Enable" "0" (at 248.92 142.24 0)
       (effects (font (size 1.27 1.27)) hide)
     )
@@
     )
   )
+  (symbol (lib_id "V2_Artwork:Socket") (at 182.88 152.4 0) (unit 1)
+    (in_bom no) (on_board yes) (dnp no) (fields_autoplaced)
+    (property "Reference" "ICON112" (at 185.42 152.4 0)
+      (effects (font (size 1.27 1.27)) (justify left))
+    )
+    (property "Value" "Socket" (at 180.34 157.48 0)
+      (effects (font (size 1.27 1.27)) (justify left bottom) hide)
+    )
+    (property "Footprint" "V2_Artwork:Socket_Small" (at 182.88 160.02 0)
+      (effects (font (size 1.27 1.27)) hide)
+    )
+    (property "Datasheet" "" (at 182.7022 152.4 0)
+      (effects (font (size 1.27 1.27)) hide)
+    )
+    (property "Sim.Enable" "0" (at 182.88 152.4 0)
+      (effects (font (size 1.27 1.27)) hide)
+    )
+    (instances
+      (project "wave"
+        (path "/6c8448b4-b04d-47e1-934e-e40cbe27a7be"
+          (reference "ICON112") (unit 1)
+        )
+      )
+    )
+  )
   (symbol (lib_id "power:GND") (at 114.3 107.95 270) (unit 1)
     (in_bom yes) (on_board yes) (dnp no)
@@
     )
   )
+  (symbol (lib_id "V2_Artwork:Dot") (at 248.92 147.32 0) (unit 1)
+    (in_bom no) (on_board yes) (dnp no) (fields_autoplaced)
+    (property "Reference" "ICON110" (at 251.46 147.32 0)
+      (effects (font (size 1.27 1.27)) (justify left))
+    )
+    (property "Value" "Dot" (at 246.38 152.4 0)
+      (effects (font (size 1.27 1.27)) (justify left bottom) hide)
+    )
+    (property "Footprint" "V2_Artwork:Dot_Small" (at 248.92 154.94 0)
+      (effects (font (size 1.27 1.27)) hide)
+    )
+    (property "Datasheet" "" (at 248.92 147.32 0)
+      (effects (font (size 1.27 1.27)) hide)
+    )
+    (property "Sim.Enable" "0" (at 248.92 147.32 0)
+      (effects (font (size 1.27 1.27)) hide)
+    )
+    (instances
+      (project "wave"
+        (path "/6c8448b4-b04d-47e1-934e-e40cbe27a7be"
+          (reference "ICON110") (unit 1)
+        )
+      )
+    )
+  )
   (symbol (lib_id "Device:R_Small") (at 138.43 53.34 90) (unit 1)
     (in_bom yes) (on_board yes) (dnp no)
@@
       (effects (font (size 1.27 1.27)) (justify left))
     )
-    (property "Value" "5k1" (at 90.6267 171.4105 0)
+    (property "Value" "2k7" (at 90.6267 171.4105 0)
       (effects (font (size 1.27 1.27)) (justify left))
     )
@@
   (sheet (at 257.81 115.57) (size 15.24 15.24) (fields_autoplaced)
     (stroke (width 0.1524) (type solid))
-    (fill (color 0 0 0 0.0000))
+    (fill (color 255 255 194 1.0000))
     (property "Sheetname" "Link Socket" (at 257.81 114.8584 0)
       (effects (font (size 1.27 1.27)) (justify left bottom))
@@
   (sheet (at 110.49 146.05) (size 21.59 39.37) (fields_autoplaced)
     (stroke (width 0.1524) (type solid))
-    (fill (color 0 0 0 0.0000))
+    (fill (color 255 255 194 1.0000))
     (property "Sheetname" "Amplifier Audio" (at 110.49 145.3384 0)
       (effects (font (size 1.27 1.27)) (justify left bottom))
@@
   (sheet (at 171.45 121.92) (size 16.51 5.08) (fields_autoplaced)
     (stroke (width 0.1524) (type solid))
-    (fill (color 0 0 0 0.0000))
+    (fill (color 255 255 194 1.0000))
     (property "Sheetname" "LED Strip" (at 171.45 121.2084 0)
       (effects (font (size 1.27 1.27)) (justify left bottom))
@@
   (sheet (at 257.81 81.28) (size 16.51 22.86)
     (stroke (width 0.1524) (type solid))
-    (fill (color 0 0 0 0.0000))
+    (fill (color 255 255 194 1.0000))
     (property "Sheetname" "Link Plug" (at 257.81 80.5684 0)
       (effects (font (size 1.27 1.27)) (justify left bottom))

Commit message: Update to Kicad 8
Parts:
- renumbered C201 to C112, C202 to C113, FB201 to FB101

Commit message: Replace icons
Parts:
- removed ICON101, ICON102, ICON104, ICON106: Minus, V2_Artwork:Minus_Small, symbol V2_Artwork:Minus
- removed ICON111: Plug, V2_Artwork:Plug_Small, symbol V2_Artwork:Plug
- removed ICON112: Socket, V2_Artwork:Socket_Small, symbol V2_Artwork:Socket
- added ICON101: Arrow_In, V2_Artwork:Arrow_In, symbol V2_Artwork:Arrow_In
- added ICON102: Arrow_Out, V2_Artwork:Arrow_Out, symbol V2_Artwork:Arrow_Out
- U101: value TPS78433QWDRBRQ1 -> TPS78433QWDRBRQ1

Commit message: Refresh
Parts:
- removed C102: 0u1, Capacitor_SMD:C_0603_1608Metric, symbol Device:C_Small
- renumbered C103 to C102, C104 to C103, C105 to C104, C106 to C105, C107 to C106, C108 to C107, C109 to C108, C110 to C109, C111 to C110, C112 to C111, C113 to C112, C114 to C113, ICON103 to ICON101, ICON107 to ICON102, ICON101 to ICON103, ICON105 to ICON104, ICON110 to ICON105, ICON102 to ICON106, ICON108 to ICON107, ICON109 to ICON108
Other:
- moved on the sheet: C101
